Commit message: simulation working well with all components with mbzirc2020_0

File: universal_robot-ur_e_fix/ur_e_description/urdf/ur5e_robot.urdf.xacro (robot description, xacro)
@@ -9,5 +9,5 @@
   <xacro:ur5e_robot parent="arm_base_frame" prefix="" joint_limited="true"/>
   <sensor_d435 parent="wrist_2_link">
-    <origin xyz="0 0 0" rpy="0 0 0"/>
+    <origin xyz="0 0 0.15" rpy="0 0 0"/>
   </sensor_d435>
   <!--

File: universal_robot-ur_e_fix/ur_e_gazebo/controller/common.gazebo.xacro (robot description, xacro)
@@ -43,5 +43,5 @@
     <plugin name="novatel_gps_sim" filename="libhector_gazebo_ros_gps.so">
       <alwaysOn>1</alwaysOn>
-      <updateRate>10.0</updateRate>
+      <updateRate>20.0</updateRate>
       <bodyName>novatel</bodyName>
       <topicName>fix</topicName>
@@ -85,5 +85,5 @@
       <plugin name="gazebo_ros_head_hokuyo_controller" filename="libgazebo_ros_laser.so">
         <topicName>scan</topicName>
-        <frameName>hokuyo</frameName>
+        <frameName>/hokuyo</frameName>
       </plugin>
     </sensor>

Commit message: Added realsense camera

File: universal_robot-ur_e_fix/ur_e_description/urdf/ur5e_robot.urdf.xacro (robot description, xacro)
@@ -7,7 +7,7 @@
   <xacro:atrvjr armConnectionFrame="arm_base_frame" prefix="${ns}"/>
   <xacro:include filename="$(find ur_e_description)/urdf/ur5e.urdf.xacro"/>
-  <xacro:include filename="$(find realsense2_description)/urdf/_d435.urdf.xacro" />
+  <xacro:include filename="$(find ur_e_description)/urdf/_d435.urdf.xacro" />
   <sensor_d435 parent="${ns}wrist_2_link" name="${ns}camera">
-    <origin xyz="0 0 0.15" rpy="0 0 0"/>
+    <origin xyz="0 0 0.15" rpy="0 0 1.5"/>
   </sensor_d435>
   <xacro:ur5e_robot parent="${ns}arm_base_frame" prefix="${ns}" joint_limited="true"/>
