Commit message: laser brick detection with execute function

File: universal_robot-ur_e_fix/ur_e_description/urdf/ur5e.urdf.xacro (robot description, xacro)
@@ -252,4 +252,17 @@
       </xacro:cylinder_inertial>
     </link>
+    <joint name="${prefix}cam_support_joint" type="fixed">
+      <parent link="${prefix}wrist_2_link" />
+      <child link = "${prefix}cam_support_link" />
+      <origin xyz="0.0 -0.05 0.2" rpy="0.0 0.0 0.0" />
+    </joint>
+    <link name="${prefix}cam_support_link">
+      <collision>
+        <geometry>
+          <box size="0.2 0.2 0.03"/>
+        </geometry>
+        <origin rpy="0 0 0" xyz="0 0 0"/>
+      </collision>
+    </link>
     <joint name="${prefix}wrist_3_joint" type="revolute">
       <parent link="${prefix}wrist_2_link" />

Commit message: Changed initial arm position

File: universal_robot-ur_e_fix/ur_e_description/urdf/ur5e.urdf.xacro (robot description, xacro)
@@ -100,5 +100,5 @@
       <parent link="${prefix}arm_base_link" />
       <child link = "${prefix}shoulder_link" />
-      <origin xyz="0.0 0.0 ${shoulder_height}" rpy="0.0 0.0 0.0" />
+      <origin xyz="0.0 0.0 ${shoulder_height}" rpy="0.0 0.0 ${pi / 2}" />
       <axis xyz="0 0 1" />
       <xacro:unless value="${joint_limited}">
@@ -131,5 +131,5 @@
       <parent link="${prefix}shoulder_link" />
       <child link = "${prefix}upper_arm_link" />
-      <origin xyz="0.0 ${shoulder_offset} 0.0" rpy="0.0 ${pi / 2.0} 0.0" />
+      <origin xyz="0.0 ${shoulder_offset} 0.0" rpy="0.0 ${pi / 4} 0.0" />
       <axis xyz="0 1 0" />
       <xacro:unless value="${joint_limited}">
@@ -162,5 +162,5 @@
       <parent link="${prefix}upper_arm_link" />
       <child link = "${prefix}forearm_link" />
-      <origin xyz="0.0 ${elbow_offset} ${upper_arm_length}" rpy="0.0 0.0 0.0" />
+      <origin xyz="0.0 ${elbow_offset} ${upper_arm_length}" rpy="0.0 ${-3 * pi / 4} 0.0" />
       <axis xyz="0 1 0" />
       <xacro:unless value="${joint_limited}">
@@ -193,5 +193,5 @@
       <parent link="${prefix}forearm_link" />
       <child link = "${prefix}wrist_1_link" />
-      <origin xyz="0.0 0.0 ${forearm_length}" rpy="0.0 ${pi / 2.0} 0.0" />
+      <origin xyz="0.0 0.0 ${forearm_length}" rpy="0.0 ${pi / 2} 0.0" />
       <axis xyz="0 1 0" />
       <xacro:unless value="${joint_limited}">
@@ -224,5 +224,5 @@
       <parent link="${prefix}wrist_1_link" />
       <child link = "${prefix}wrist_2_link" />
-      <origin xyz="0.0 ${wrist_1_length} 0.0" rpy="0.0 0.0 0.0" />
+      <origin xyz="0.0 ${wrist_1_length} 0.0" rpy="0.0 0.0 ${pi / 2}" />
       <axis xyz="0 0 1" />
       <xacro:unless value="${joint_limited}">
