Commit message: major changes to namespace. working version with atrvjr namespace

File: atrvjr/description/atrvjr_description/urdf/atrvjr.xacro (robot description, xacro)
@@ -1,5 +1,5 @@
 <?xml version="1.0"?>
 <robot xmlns:xacro="http://www.ros.org/wiki/xacro" name="atrvjr">
-    <xacro:macro name="atrvjr" params="armConnectionFrame">
+    <xacro:macro name="atrvjr" params="armConnectionFrame prefix">
     <xacro:property name="M_PI" value="3.14159"/>
     <!-- Robot parameters -->
@@ -18,16 +18,16 @@
     <xacro:property name="wheel_long_offset" value="0.19 " /> <!-- distance from robot center to wheel center in x direction (forward direction) -->
     <xacro:property name="wheel_lat_offset" value="0.25" /> <!-- distance from robot center to wheel center in y direction (lateral direction) -->
-    <xacro:include filename="$(find atrvjr_description)/urdf/atrvjr_wheels.xacro" />
+    <xacro:include filename="$(find atrvjr_description)/urdf/atrvjr_wheels.xacro"/>
     <!-- mbot wheel generation based on imported macro -->
-    <xacro:wheel prefix="front" side="left" origin_x="${wheel_long_offset}" origin_y="${wheel_lat_offset}" >
+    <xacro:wheel prefix="${prefix}front" side="left" origin_x="${wheel_long_offset}" origin_y="${wheel_lat_offset}" parent="${prefix}base_link" >
         <origin xyz="0 0 0" rpy="0 0 0" />
     </xacro:wheel>
-    <xacro:wheel prefix="front" side="right" origin_x="${wheel_long_offset}" origin_y="-${wheel_lat_offset}" >
+    <xacro:wheel prefix="${prefix}front" side="right" origin_x="${wheel_long_offset}" origin_y="-${wheel_lat_offset}" parent="${prefix}base_link" >
         <origin xyz="0 0 0" rpy="0 0 0" />
     </xacro:wheel>
-    <xacro:wheel prefix="rear" side="left" origin_x="-${wheel_long_offset}" origin_y="${wheel_lat_offset}" >
+    <xacro:wheel prefix="${prefix}rear" side="left" origin_x="-${wheel_long_offset}" origin_y="${wheel_lat_offset}" parent="${prefix}base_link" >
         <origin xyz="0 0 0" rpy="0 0 0" />
     </xacro:wheel>
-    <xacro:wheel prefix="rear" side="right" origin_x="-${wheel_long_offset}" origin_y="-${wheel_lat_offset}" >
+    <xacro:wheel prefix="${prefix}rear" side="right" origin_x="-${wheel_long_offset}" origin_y="-${wheel_lat_offset}" parent="${prefix}base_link" >
         <origin xyz="0 0 0" rpy="0 0 0" />
     </xacro:wheel>
@@ -72,5 +72,5 @@
     <!-- The frame of the floor directly below the center_link and -->
     <!-- is needed for the navigation stack to work properly -->
-    <link name="base_link">
+    <link name="${prefix}base_link">
         <inertial>
             <origin xyz="0.0 0.0 0.2" rpy="0 0 0"/>
@@ -83,5 +83,5 @@
     <!-- robot and should also represent the main chassis via inertial, -->
     <!-- visual, and geometry elements of the link -->
-    <link name="center_link">
+    <link name="${prefix}center_link">
         <visual>
             <geometry>
@@ -97,37 +97,37 @@
     </link>
     <!-- base_link -> center_link -->
-    <joint name="base_link_joint" type="fixed">
+    <joint name="${prefix}base_link_joint" type="fixed">
         <origin xyz="-0.1 0.19 ${center_height-0.1}" rpy="1.57 0 0"/>
-        <parent link="base_link"/>
-        <child link="center_link"/>
+        <parent link="${prefix}base_link"/>
+        <child link="${prefix}center_link"/>
     </joint>
      <!-- Arm Link -->
-    <link name="${armConnectionFrame}"/>
-    <joint name="$to_{armConnectionFrame}_joint" type="fixed">
+    <link name="${prefix}${armConnectionFrame}"/>
+    <joint name="${prefix}$to_{armConnectionFrame}_joint" type="fixed">
         <origin xyz="0.09 0 0.47" rpy="0 0 0"/>
-        <parent link="base_link"/>
-        <child link="${armConnectionFrame}"/>
+        <parent link="${prefix}base_link"/>
+        <child link="${prefix}${armConnectionFrame}"/>
     </joint>
     <!-- Crossbow Imu Link -->
-    <link name="cbimu_frame"/>
-    <joint name="base_cbimu_joint" type="fixed">
+    <link name="${prefix}cbimu_frame"/>
+    <joint name="${prefix}base_cbimu_joint" type="fixed">
         <origin xyz="0 0 0.267" rpy="0 ${M_PI} 0"/>
-        <parent link="base_link"/>
-        <child link="cbimu_frame"/>
+        <parent link="${prefix}base_link"/>
+        <child link="${prefix}cbimu_frame"/>
     </joint>
         <!-- MPU Imu Link -->
-    <link name="mpuimu_frame"/>
-    <joint name="base_mpuimu_joint" type="fixed">
+    <link name="${prefix}mpuimu_frame"/>
+    <joint name="${prefix}base_mpuimu_joint" type="fixed">
         <origin xyz="0 -0.1 0.55" rpy="0 0 0"/>
-        <parent link="base_link"/>
-        <child link="mpuimu_frame"/>
+        <parent link="${prefix}base_link"/>
+        <child link="${prefix}mpuimu_frame"/>
     </joint>
-    <link name="novatel"/>
-    <joint name="novatel_joint" type="fixed">
+    <link name="${prefix}novatel"/>
+    <joint name="${prefix}novatel_joint" type="fixed">
         <origin xyz="-0.15 0.1 0.55" rpy="0 0 0"/>
-        <parent link="base_link"/>
-        <child link="novatel"/>
+        <parent link="${prefix}base_link"/>
+        <child link="${prefix}novatel"/>
     </joint>
-    <link name="hokuyo"/>
+    <link name="${prefix}hokuyo"/>
 <!--         <visual>
             <geometry>
@@ -141,8 +141,8 @@
         </inertial>
     </link> -->
-    <joint name="laser_joint" type="fixed">
+    <joint name="${prefix}laser_joint" type="fixed">
         <origin xyz="0.37 0 0.135" rpy="${M_PI} 0 0"/>
-        <parent link="base_link" />
-        <child link="hokuyo" />
+        <parent link="${prefix}base_link" />
+        <child link="${prefix}hokuyo" />
     </joint>
    <!--  <transmission name="teste_prismatic_trans">

File: atrvjr/description/atrvjr_description/urdf/atrvjr_wheels.xacro (robot description, xacro)
@@ -2,5 +2,5 @@
 <robot xmlns:xacro="http://wiki.ros.org/xacro" name="atrvjr" >
   <!-- wheel macro -->
-  <xacro:macro name="wheel" params="prefix side origin_x origin_y *joint_pose">
+  <xacro:macro name="wheel" params="prefix side origin_x origin_y *joint_pose parent">
     <!-- dummy link from which the real wheel will rotate from -->
     <link name="${prefix}_${side}_static">
@@ -16,5 +16,5 @@
     <!-- to specify the position of the dummy link w.r.t. base link -->
     <joint name="${prefix}_${side}_static_joint" type="fixed">
-      <parent link="base_link"/>
+      <parent link="${parent}"/>
       <child link="${prefix}_${side}_static" />
       <origin xyz="${origin_x} ${origin_y} ${wheel_radius}" rpy="0 0 0" />

File: universal_robot-ur_e_fix/ur_e_description/urdf/ur5e_robot.urdf.xacro (robot description, xacro)
@@ -2,13 +2,14 @@
 <robot xmlns:xacro="http://ros.org/wiki/xacro"
        name="atrv_ur5e" >
+  <xacro:property name="ns" value="atrvjr/" />
   <xacro:include filename="$(find ur_e_gazebo)/controller/common.gazebo.xacro" />
   <xacro:include filename="$(find atrvjr_description)/urdf/atrvjr.xacro"/>
-  <xacro:atrvjr armConnectionFrame="arm_base_frame"/>
-  <xacro:include filename="$(find ur_e_description)/urdf/ur5e.urdf.xacro" />
-  <xacro:include filename="$(find realsense2_description)/urdf/_d435.urdf.xacro"/>
-  <xacro:ur5e_robot parent="arm_base_frame" prefix="" joint_limited="true"/>
-  <sensor_d435 parent="wrist_2_link">
+  <xacro:atrvjr armConnectionFrame="arm_base_frame" prefix="${ns}"/>
+  <xacro:include filename="$(find ur_e_description)/urdf/ur5e.urdf.xacro"/>
+  <xacro:include filename="$(find realsense2_description)/urdf/_d435.urdf.xacro" />
+  <sensor_d435 parent="${ns}wrist_2_link" name="${ns}camera">
     <origin xyz="0 0 0.15" rpy="0 0 0"/>
   </sensor_d435>
+  <xacro:ur5e_robot parent="${ns}arm_base_frame" prefix="${ns}" joint_limited="true"/>
   <!--
   <link name="world" /> -->

File: universal_robot-ur_e_fix/ur_e_gazebo/controller/common.gazebo.xacro (robot description, xacro)
@@ -3,5 +3,5 @@
   <gazebo>
     <plugin name="ros_control" filename="libgazebo_ros_control.so">
-      <robotNamespace>/mbzirc2020_0</robotNamespace>
+      <!-- <robotNamespace>/mbzirc2020_0</robotNamespace> -->
       <robotSimType>gazebo_ros_control/DefaultRobotHWSim</robotSimType>
       <legacyModeNS>true</legacyModeNS>
@@ -44,5 +44,5 @@
       <alwaysOn>1</alwaysOn>
       <updateRate>20.0</updateRate>
-      <bodyName>novatel</bodyName>
+      <bodyName>atrvjr/novatel</bodyName>
       <topicName>fix</topicName>
       <velocityTopicName>fix_velocity</velocityTopicName>

Commit message: created a simulation branch closer to reality. Double EKF simulation available

File: atrvjr/description/atrvjr_description/urdf/atrvjr.xacro (robot description, xacro)
@@ -109,17 +109,10 @@
         <child link="${prefix}${armConnectionFrame}"/>
     </joint>
-    <!-- Crossbow Imu Link -->
-    <link name="${prefix}cbimu_frame"/>
-    <joint name="${prefix}base_cbimu_joint" type="fixed">
-        <origin xyz="0 0 0.267" rpy="0 ${M_PI} 0"/>
+        <!-- pixhawk Imu Link -->
+    <link name="${prefix}pixhawkimu_frame"/>
+    <joint name="${prefix}base_pixhawkimu_joint" type="fixed">
+        <origin xyz="0 0.0 0.55" rpy="0 0 0"/>
         <parent link="${prefix}base_link"/>
-        <child link="${prefix}cbimu_frame"/>
-    </joint>
-        <!-- MPU Imu Link -->
-    <link name="${prefix}mpuimu_frame"/>
-    <joint name="${prefix}base_mpuimu_joint" type="fixed">
-        <origin xyz="0 -0.1 0.55" rpy="0 0 0"/>
-        <parent link="${prefix}base_link"/>
-        <child link="${prefix}mpuimu_frame"/>
+        <child link="${prefix}pixhawkimu_frame"/>
     </joint>
     <link name="${prefix}novatel"/>

File: universal_robot-ur_e_fix/ur_e_gazebo/controller/common.gazebo.xacro (robot description, xacro)
@@ -22,18 +22,18 @@
 -->
   </gazebo>
-<gazebo reference="mpuimu_frame">
+<gazebo reference="atrvjr/pixhawkimu_frame">
     <gravity>true</gravity>
-    <sensor name="mpu_imu" type="imu">
+    <sensor name="pixhawk_imu" type="imu">
         <always_on>true</always_on>
         <update_rate>100</update_rate>
-        <topic>/imu</topic>
+        <topic>pixhawkimu/data</topic>
         <plugin filename="libgazebo_ros_imu_sensor.so" name="imu_plugin">
-            <topicName>/imu/data</topicName>
-            <bodyName>mpuimu_frame</bodyName>
+            <topicName>pixhawkimu/data</topicName>
+            <bodyName>atrvjr/pixhawkimu_frame</bodyName>
             <updateRateHZ>100</updateRateHZ>
             <gaussianNoise>0.0</gaussianNoise>
             <xyzOffset>0 0 0</xyzOffset>
             <rpyOffset>0 0 0</rpyOffset>
-            <frameName>mpuimu_frame</frameName>
+            <frameName>atrvjr/pixhawkimu_frame</frameName>
         </plugin>
         <pose>0 0 0 0 0 0</pose>
@@ -46,4 +46,6 @@
       <bodyName>atrvjr/novatel</bodyName>
       <topicName>fix</topicName>
+      <referenceLatitude>38.540272</referenceLatitude>
+      <referenceLongitude>-7.962953</referenceLongitude>
       <velocityTopicName>fix_velocity</velocityTopicName>
       <drift>0 0 0</drift>

Commit message: Ajusted navigation parameters for both robots

File: atrvjr/description/atrvjr_description/urdf/atrvjr.xacro (robot description, xacro)
@@ -123,4 +123,10 @@
         <child link="${prefix}mpuimu_frame"/>
     </joint>
+    <link name="${prefix}imu_link"/>
+    <joint name="${prefix}imu_joint" type="fixed">
+        <origin xyz="0.0 0.0 0.0" rpy="0 0 0"/>
+        <parent link="${prefix}base_link"/>
+        <child link="${prefix}imu_link"/>
+    </joint>
     <link name="${prefix}novatel"/>
     <joint name="${prefix}novatel_joint" type="fixed">

File: universal_robot-ur_e_fix/ur_e_gazebo/controller/common.gazebo.xacro (robot description, xacro)
@@ -22,5 +22,5 @@
 -->
   </gazebo>
-<gazebo reference="mpuimu_frame">
+<!-- <gazebo reference="mpuimu_frame">
     <gravity>true</gravity>
     <sensor name="mpu_imu" type="imu">
@@ -29,5 +29,5 @@
         <topic>/imu</topic>
         <plugin filename="libgazebo_ros_imu_sensor.so" name="imu_plugin">
-            <topicName>/imu/data</topicName>
+            <topicName>atrvjr/imu/data</topicName>
             <bodyName>mpuimu_frame</bodyName>
             <updateRateHZ>100</updateRateHZ>
@@ -39,5 +39,20 @@
         <pose>0 0 0 0 0 0</pose>
     </sensor>
-</gazebo>
+</gazebo> -->
+<gazebo>
+    <plugin name="imu_controller" filename="libhector_gazebo_ros_imu.so">
+      <robotNamespace>/atrvjr</robotNamespace>
+      <updateRate>50.0</updateRate>
+      <bodyName>atrvjr/imu_link</bodyName>
+      <topicName>imu/data</topicName>
+      <frameId>imu_link</frameId>
+      <accelDrift>0.00 0.00 0.00</accelDrift>
+      <accelGaussianNoise>0.001 0.001 0.001</accelGaussianNoise>
+      <rateDrift>0.00 0.00 0.00 </rateDrift>
+      <rateGaussianNoise>0.001 0.001 0.001 </rateGaussianNoise>
+      <headingDrift>0.00</headingDrift>
+      <headingGaussianNoise>0.001</headingGaussianNoise>
+    </plugin>
+  </gazebo>
  <gazebo>
     <plugin name="novatel_gps_sim" filename="libhector_gazebo_ros_gps.so">
